File: UselessBox.sch (EAGLE design)
At the start: 20 parts, among them Q2 MJE182-VERTICAL, U2 5V, X1 SCREW-TERM-3, X2 SCREW-TERM-3

Commit message: Update size of bypass caps
Parts:
- C1, C2: device SaintGimp:CAPACITOR-2.5MM -> SaintGimp:CAPACITOR-5MM
Changed lines of the file:
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@@
 <layer number="97" name="Info" color="7" fill="1" visible="yes" active="yes"/>
 <layer number="98" name="Guide" color="6" fill="1" visible="yes" active="yes"/>
+<layer number="99" name="SpiceOrder" color="7" fill="1" visible="yes" active="yes"/>
 <layer number="100" name="Muster" color="7" fill="1" visible="no" active="no"/>
 <layer number="101" name="Patch_Top" color="12" fill="4" visible="yes" active="yes"/>
@@
 <layer number="111" name="LPC17xx" color="7" fill="1" visible="yes" active="yes"/>
 <layer number="112" name="tSilk" color="7" fill="1" visible="yes" active="yes"/>
+<layer number="113" name="IDFDebug" color="7" fill="1" visible="yes" active="yes"/>
 <layer number="116" name="Patch_BOT" color="9" fill="4" visible="yes" active="yes"/>
 <layer number="121" name="_tsilk" color="7" fill="1" visible="yes" active="yes"/>
@@
 <layer number="251" name="SMDround" color="7" fill="1" visible="no" active="no"/>
 <layer number="254" name="cooling" color="7" fill="1" visible="yes" active="yes"/>
+<layer number="255" name="routoute" color="7" fill="1" visible="yes" active="yes"/>
 </layers>
 <schematic xreflabel="%F%N/%S.%C%R" xrefpart="/%S.%C%R">
@@
 <part name="ATMEGA328P" library="SaintGimp" deviceset="ATMEGA328P-PU" device=""/>
 <part name="GND1" library="supply1" deviceset="GND" device=""/>
-<part name="C1" library="SaintGimp" deviceset="CAPACITOR-*" device="2.5MM" value="1uF"/>
-<part name="C2" library="SaintGimp" deviceset="CAPACITOR-*" device="2.5MM" value="1uF"/>
+<part name="C1" library="SaintGimp" deviceset="CAPACITOR-*" device="5MM" value="1uF"/>
+<part name="C2" library="SaintGimp" deviceset="CAPACITOR-*" device="5MM" value="1uF"/>
 <part name="GND2" library="supply1" deviceset="GND" device=""/>
 <part name="GND3" library="supply1" deviceset="GND" device=""/>

Commit message: Update parts from library
Parts:
- Q2: value MJE182-VERTICAL -> MJE182-V; device SaintGimp:MJE182-VERTICAL -> SaintGimp:MJE182-V
Changed lines of the file:
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@@
 <part name="C6" library="SaintGimp" deviceset="CAP-POL" device="-5-10" value="2200uF"/>
 <part name="GND9" library="supply1" deviceset="GND" device=""/>
-<part name="Q2" library="SaintGimp" deviceset="MJE182-*" device="VERTICAL"/>
+<part name="Q2" library="SaintGimp" deviceset="MJE182" device="-V"/>
 <part name="GND5" library="supply1" deviceset="GND" device=""/>
 <part name="X1" library="SaintGimp" deviceset="SCREW-TERM-3" device=""/>
